File: lol/lol.sch (KiCad schematic (older format))
At the start: 20 parts, among them J1 USB_B_Micro, J2 5V_BUS, J3 GP_IO, SW1 SW_Push, SW2 SW_Push, SW3 SW_Push, U1 ATmega32U4-MU, Y1 16MHz

Commit message: update
Parts:
- added D4: LED, LED_THT:LED_D4.0mm, symbol Device:LED
- added R7: R, Resistor_THT:R_Axial_DIN0204_L3.6mm_D1.6mm_P5.08mm_Horizontal, symbol Device:R
- SW1, SW2, SW3: footprint Button_Switch_Keyboard:SW_Cherry_MX_1.00u_PCB -> Button_Switch_THT:SW_PUSH_6mm
Connections:
- net GND: now also D4.1 (K)
- net LED1: now reaches U1.21 (PD3)
- net LED1: now also R7.1
- new net: D4.2 (A), R7.2
- no-connect marks 17 -> 16
Other:
- note added: "Crystal, generates clock \nsignal for microcontroller\n"
- note added: "Fuse limits current draw"
- note added: "Micro USB Port"
- moved on the sheet: C1, C2, C3, C4, F1, J1, J2, R1, R2
